Commit message: Edited parameters during test. Modified launch files. Added maps.

File: paprika_description/urdf/paprika_simple.xacro (robot description, xacro)
@@ -11,5 +11,5 @@
   <parent link="chassis"/>
   <child link="camera_link"/>
-    <origin xyz="0 0.045 0.3075" rpy="0 0 0"/>
+    <origin xyz="0.17 0.045 0.0525" rpy="0 0 0"/>
 </joint>
 <link name = "camera_link" />
