Commit message: Added Rviz during launch. Modified URDF file for the new chassis.

File: paprika_description/urdf/paprika_old.xacro (robot description, xacro)
@@ -5,5 +5,5 @@
   <parent link="base_link"/>
   <child link="chassis"/>
-    <origin xyz="0 0 0.10" rpy="0 0 0"/>
+    <origin xyz="0 0 0.105" rpy="0 0 0"/>
 </joint>
 <link name = "chassis" />
@@ -11,5 +11,5 @@
   <parent link="chassis"/>
   <child link="camera_link"/>
-    <origin xyz="0.16 0.045 0.415" rpy="0 0 0"/>
+    <origin xyz="0.17 0.045 0.0525" rpy="0 0 0"/>
 </joint>
 <link name = "camera_link" />
